File: hardware/destinationWeatherStation_r4-5.kicad_pcb (KiCad board)
At the start: 2 copper layers, 63.5 x 50.8 mm, 39 parts, among them J1 S2B-PH-SM4, J2 MEM2061, J3 STEMMA_QT, Q1 IRLML6244TRPBF, Q2 IRLML6244TRPBF, Q3 DMP2035UVTQ-7, Q4 DMP2035UVTQ-7, SW1 SS-12F44-G5, SW2 PTS647SM38SMTR2LFS, SW3 PTS647SM38SMTR2LFS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

Commit message: blender stuff
Other:
- board text added: "PCB3D_BR_DSWXSTN4-5"
- board text added: "PCB3D_TL_DSWXSTN4-5"
Changed lines of the file:
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@@
       (layer "F.SilkS" (type "Top Silk Screen") (color "White") (material "Direct Printing"))
       (layer "F.Paste" (type "Top Solder Paste"))
-      (layer "F.Mask" (type "Top Solder Mask") (color "Black") (thickness 0.0254) (material "Liquid Ink") (epsilon_r 3.8) (loss_tangent 0))
+      (layer "F.Mask" (type "Top Solder Mask") (color "Purple") (thickness 0.0254) (material "Liquid Ink") (epsilon_r 3.8) (loss_tangent 0))
       (layer "F.Cu" (type "copper") (thickness 0.035))
       (layer "dielectric 1" (type "core") (color "FR4 natural") (thickness 1.4292) (material "FR408-HR") (epsilon_r 4.7) (loss_tangent 0.0091))
       (layer "B.Cu" (type "copper") (thickness 0.035))
-      (layer "B.Mask" (type "Bottom Solder Mask") (color "Black") (thickness 0.0254) (material "Liquid Ink") (epsilon_r 3.8) (loss_tangent 0))
+      (layer "B.Mask" (type "Bottom Solder Mask") (color "Purple") (thickness 0.0254) (material "Liquid Ink") (epsilon_r 3.8) (loss_tangent 0))
       (layer "B.Paste" (type "Bottom Solder Paste"))
       (layer "B.SilkS" (type "Bottom Silk Screen") (color "White") (material "Direct Printing"))
@@
     )
   )
+  (gr_text "PCB3D_TL_DSWXSTN4-5" (at 113.03 71.12) (layer "Cmts.User")
+    (effects (font (size 1 1) (thickness 0.15)) (justify right bottom))
+  )
+  (gr_text "PCB3D_BR_DSWXSTN4-5" (at 176.53 121.92) (layer "Cmts.User")
+    (effects (font (size 1 1) (thickness 0.15)) (justify left bottom))
+  )
   (gr_text_box "Destination SPACE Inc.\nDesigned in Asheville, NC\nby Madison Gleydura"
