File: hardware/destinationWeatherStation_r4-5.kicad_pcb (KiCad board)
At the start: 2 copper layers, 63.5 x 50.8 mm, 39 parts, among them J1 S2B-PH-SM4, J2 MEM2061, J3 STEMMA_QT, Q1 IRLML6244TRPBF, Q2 IRLML6244TRPBF, Q3 DMP2035UVTQ-7, Q4 DMP2035UVTQ-7, SW1 SS-12F44-G5, SW2 PTS647SM38SMTR2LFS, SW3 PTS647SM38SMTR2LFS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

Commit message: finalized PCB CAD
Parts:
- JP1, JP2: footprint lib_fp:SolderJumper-3_P1.3mm_Open_RoundedPad1.0x1.5mm -> lib_fp:ResistorJumper-3
- moved C2 0.27 mm to (130.6, 118.4)
- moved C1 0.18 mm to (130.6, 115.3)
Other:
- board text added: "Destination Weather Station v4.5.2 2024-02-12"
- board text added: "Student Name:"
- board text removed: "Destination Weather Station v4.5.1 2024-01-07"
- board text removed: "Name:"

Commit message: file touchups
Parts:
- removed JP1, JP2: Jumper_3_Open, lib_fp:ResistorJumper-3
- added R11: 0R, lib_fp:ResistorJumper-3, F.Cu at (152.4, 87.0)
- added R12: 0R, lib_fp:ResistorJumper-3, F.Cu at (154.9, 87.0)

Commit message: changes
Parts:
- removed kibuzzard-64039D84: G***, lib_fp:kibuzzard-64039D84
- removed kibuzzard-64039D9C: G***, lib_fp:kibuzzard-64039D9C
- added G***: LOGO, DS-Master-Logos-and-Graphics:arrow, F.Cu at (156.3, 88.0)
- added G***: LOGO, DS-Master-Logos-and-Graphics:arrow, F.Cu at (151.1, 86.0)
Routing:
- net GND: track 19.1 -> 16.6 mm, vias 21 -> 221
- added copper zone on F.Cu, net +3V3
Other:
- board text added: "Destination Weather Station v4.5.2 2024-02-22"
- board text added: "OFF"
- board text added: "ON"
- board text added: "PCB3D_BR_DS-WX-STN-v4-5"
- board text added: "PCB3D_TL_DS-WX-STN-v4-5"
- board text removed: "Destination Weather Station v4.5.2 2024-02-12"
