File: hardware/destinationWeatherStation_r4-5.kicad_pcb (KiCad board)
At the start: 2 copper layers, 63.5 x 50.8 mm, 39 parts, among them J1 S2B-PH-SM4, J2 MEM2061, J3 STEMMA_QT, Q1 IRLML6244TRPBF, Q2 IRLML6244TRPBF, Q3 DMP2035UVTQ-7, Q4 DMP2035UVTQ-7, SW1 SS-12F44-G5, SW2 PTS647SM38SMTR2LFS, SW3 PTS647SM38SMTR2LFS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

Commit message: 3d pdf stuff and board fixes
Routing:
- net +3V3: track 197.6 -> 186.0 mm
- net /MOSI: track 36.7 -> 41.2 mm, vias 3 -> 2
- net /SW3: track 78.3 -> 74.5 mm, vias 1 -> 0
- net /SCL: track 78.7 -> 82.3 mm, vias 3 -> 4
- net /SDA: track 89.7 -> 91.0 mm, vias 3 -> 4
- net /SW2: track 60.6 -> 59.5 mm, vias 1 -> 0
- net /SW4: track 65.0 -> 65.9 mm
- net GND: vias 221 -> 222
Other:
- board text added: "Destination Weather Station v4.5.2 2024-02-23"
- board text removed: "Destination Weather Station v4.5.2 2024-02-22"

Commit message: final CAD changes
Routing:
- net GND: track 16.6 -> 15.5 mm, vias 222 -> 223
Other:
- board text added: "Destination Weather Station v4.5.2 2024-02-24"
- board text removed: "Destination Weather Station v4.5.2 2024-02-23"
