File: hardware/destinationWeatherStation_r4-5.kicad_sch (KiCad schematic)
At the start: 35 parts, among them J1 S2B-PH-SM4, J2 MEM2061, J3 STEMMA_QT, Q1 IRLML6244TRPBF, Q2 IRLML6244TRPBF, Q3 DMP2035UVTQ-7, Q4 DMP2035UVTQ-7, SW1 SS-12F44-G5, SW2 PTS647SM38SMTR2LFS, U1 XIAO RP2040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

Commit message: finalized PCB CAD
Parts:
- JP1, JP2: footprint lib_fp:SolderJumper-3_P1.3mm_Open_RoundedPad1.0x1.5mm -> lib_fp:ResistorJumper-3; Manufacturer (none) -> Vishay Dale; mpn (none) -> CRCW06030000Z0EA; populate 0 -> 1
- R1, R10, R2, R3, R4, R5, R6, R7, R8, R9: populate (none) -> 1
Other:
- title: Destination Weather Station R4 -> Destination Weather Station v4.5.2

Commit message: file touchups
Parts:
- removed JP1, JP2: Jumper_3_Open, lib_fp:ResistorJumper-3, symbol lib_sch:Jumper_3_Open
- added R11, R12: 0R, lib_fp:ResistorJumper-3, symbol lib_sch:Resistor_Jumper_3_Open
Connections:
- net +3V3: now also R11.1 (A), R12.3 (B)
- net GND: now also R11.3 (B), R12.1 (A)
- net OLED1: now also R11.2 (C)
- net OLED2: now also R12.2 (C)
Changed lines of the file:
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@@
   (title_block
     (title "Destination Weather Station v4.5.2")
-    (date "2024-02-12")
-    (rev "02")
+    (date "2024-02-16")
+    (rev "03")
     (comment 1 "Madison Gleydura")
     (comment 2 "FINAL VERSION")
@@
     )
   )
+  (symbol (lib_id "lib_sch:Resistor_Jumper_3_Open") (at 125.73 116.84 0) (unit 1)
+    (in_bom yes) (on_board yes) (dnp no)
+    (property "Reference" "R11" (at 125.73 114.3 0)
+      (effects (font (size 1.27 1.27)))
+    )
+    (property "Value" "0R" (at 125.73 113.03 0)
+      (effects (font (size 1.27 1.27)) hide)
+    )
+    (property "Footprint" "lib_fp:ResistorJumper-3" (at 125.73 116.84 0)
+      (effects (font (size 1.27 1.27)) hide)
+    )
+    (property "Datasheet" "datasheets/Vishay-Dale-DCRCWe3.pdf" (at 125.73 116.84 0)
+      (effects (font (size 1.27 1.27)) hide)
+    )
+    (property "Manufacturer" "Vishay Dale" (at 125.73 116.84 0)
+      (effects (font (size 1.27 1.27)) hide)
+    )
+    (property "mpn" "CRCW06030000Z0EA" (at 125.73 116.84 0)
+      (effects (font (size 1.27 1.27)) hide)
+    )
+    (property "populate" "1" (at 125.73 116.84 0)
+      (effects (font (size 1.27 1.27)) hide)
+    )
+    (pin "2")
+    (pin "1")
+    (pin "3")
+    (instances
+      (project "destinationWeatherStation_r4-5"
+        (path "/ee9b83c5-5ca5-4f3a-b6eb-6165828355bc"
+          (reference "R11") (unit 1)
+        )
+      )
+    )
+  )
   (symbol (lib_id "power:+3V3") (at 46.99 191.77 0) (mirror y) (unit 1)
     (in_bom yes) (on_board yes) (dnp no)
@@
         (path "/ee9b83c5-5ca5-4f3a-b6eb-6165828355bc"
           (reference "R3") (unit 1)
+        )
+      )
+    )
+  )
+  (symbol (lib_id "lib_sch:Resistor_Jumper_3_Open") (at 143.51 116.84 0) (unit 1)
+    (in_bom yes) (on_board yes) (dnp no)
+    (property "Reference" "R12" (at 143.51 114.3 0)
+      (effects (font (size 1.27 1.27)))
+    )
+    (property "Value" "0R" (at 143.51 113.03 0)
+      (effects (font (size 1.27 1.27)) hide)
+    )
+    (property "Footprint" "lib_fp:ResistorJumper-3" (at 143.51 116.84 0)
+      (effects (font (size 1.27 1.27)) hide)
+    )
+    (property "Datasheet" "datasheets/Vishay-Dale-DCRCWe3.pdf" (at 143.51 116.84 0)
+      (effects (font (size 1.27 1.27)) hide)
+    )
+    (property "Manufacturer" "Vishay Dale" (at 143.51 116.84 0)
+      (effects (font (size 1.27 1.27)) hide)
+    )
+    (property "mpn" "CRCW06030000Z0EA" (at 143.51 116.84 0)
+      (effects (font (size 1.27 1.27)) hide)
+    )
+    (property "populate" "1" (at 143.51 116.84 0)
+      (effects (font (size 1.27 1.27)) hide)
+    )
+    (pin "2")
+    (pin "1")
+    (pin "3")
+    (instances
+      (project "destinationWeatherStation_r4-5"
+        (path "/ee9b83c5-5ca5-4f3a-b6eb-6165828355bc"
+          (reference "R12") (unit 1)
         )
       )
@@
     )
   )
-  (symbol (lib_id "lib_sch:Jumper_3_Open") (at 125.73 116.84 0) (unit 1)
-    (in_bom yes) (on_board yes) (dnp no)
-    (property "Reference" "JP1" (at 125.73 110.49 0)
-      (effects (font (size 1.27 1.27)))
-    )
-    (property "Value" "Jumper_3_Open" (at 125.73 113.03 0)
-      (effects (font (size 1.27 1.27)))
-    )
-    (property "Footprint" "lib_fp:ResistorJumper-3" (at 125.73 116.84 0)
-      (effects (font (size 1.27 1.27)) hide)
-    )
-    (property "Datasheet" "datasheets/Vishay-Dale-DCRCWe3.pdf" (at 125.73 116.84 0)
-      (effects (font (size 1.27 1.27)) hide)
-    )
-    (property "Manufacturer" "Vishay Dale" (at 125.73 116.84 0)
-      (effects (font (size 1.27 1.27)) hide)
-    )
-    (property "mpn" "CRCW06030000Z0EA" (at 125.73 116.84 0)
-      (effects (font (size 1.27 1.27)) hide)
-    )
-    (property "populate" "1" (at 125.73 116.84 0)
-      (effects (font (size 1.27 1.27)) hide)
-    )
-    (pin "1")
-    (pin "2")
-    (pin "3")
-    (instances
-      (project "destinationWeatherStation_r4-5"
-        (path "/ee9b83c5-5ca5-4f3a-b6eb-6165828355bc"
-          (reference "JP1") (unit 1)
-        )
-      )
-    )
-  )
   (symbol (lib_id "lib_sch:r_small") (at 199.39 24.13 0) (unit 1)
     (in_bom yes) (on_board yes) (dnp no)
@@
         )
       )
-    )
-  )
-  (symbol (lib_id "lib_sch:Jumper_3_Open") (at 143.51 116.84 0) (mirror y) (unit 1)
-    (in_bom yes) (on_board yes) (dnp no)
-    (property "Reference" "JP2" (at 143.51 110.49 0)
-      (effects (font (size 1.27 1.27)))
-    )
-    (property "Value" "Jumper_3_Open" (at 143.51 113.03 0)
-      (effects (font (size 1.27 1.27)))
-    )
-    (property "Footprint" "lib_fp:ResistorJumper-3" (at 143.51 116.84 0)
-      (effects (font (size 1.27 1.27)) hide)
-    )
-    (property "Datasheet" "datasheets/Vishay-Dale-DCRCWe3.pdf" (at 143.51 116.84 0)
-      (effects (font (size 1.27 1.27)) hide)
-    )
-    (property "Manufacturer" "Vishay Dale" (at 143.51 116.84 0)
-      (effects (font (size 1.27 1.27)) hide)
-    )
-    (property "mpn" "CRCW06030000Z0EA" (at 143.51 116.84 0)
-      (effects (font (size 1.27 1.27)) hide)
-    )
-    (property "populate" "1" (at 143.51 116.84 0)
-      (effects (font (size 1.27 1.27)) hide)
-    )
-    (pin "1")
-    (pin "2")
-    (pin "3")
-    (instances
-      (project "destinationWeatherStation_r4-5"
-        (path "/ee9b83c5-5ca5-4f3a-b6eb-6165828355bc"
-          (reference "JP2") (unit 1)
-        )
-      )

Commit message: changes
Other:
- note added: "M2.5 Mounting Holes"
- note added: "STEMMA QT Connector"
- note removed: "M3 Mounting Holes"
- moved on the sheet: C1, C2, J3, R11, R12, U1, U3

Commit message: 3d pdf stuff and board fixes
Other:
- note added: "OLED Display"
- note removed: "OLED"
- moved on the sheet: J2, R1, R2, R3, R4, R5, R6, R7, SW2, U1

Commit message: fixes
Parts:
- C1: mpn KGM15CR51A106MT -> KGM15CR51A106KT
Changed lines of the file:
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@@
       (effects (font (size 1.27 1.27)) hide)
     )
-    (property "mpn" "KGM15CR51A106MT" (at 152.4 22.225 0)
+    (property "mpn" "KGM15CR51A106KT" (at 152.4 22.225 0)
       (effects (font (size 1.27 1.27)) hide)
     )

Commit message: test jig code
Other:
- note added: "ADDR: 0x76"
Changed lines of the file:
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@@
+    (effects (font (size 1.27 1.27)) (justify left bottom))
+  )
+  (text "ADDR: 0x76" (at 44.45 138.43 0)
     (effects (font (size 1.27 1.27)) (justify left bottom))
   )
